Commit message: construct urdf object from Jinja template

File: models/quadruped.urdf (robot description, URDF)
Before this commit: robot {{ name }}, 2 links, 1 joints
Links:
- removed link body
- removed link {{ appendage }}
- added link {{ name }}, mass {{ component.mass }}; collision mesh filename={{ component.model }} scale={{ scale }} {{ scale }} {{ scale }}; visual mesh filename={{ component.model }} scale={{ scale }} {{ scale }} {{ scale }}
Joints:
- removed joint {{ joint.name }}
- added joint {{ parent }}-{{ child }}: type revolute, parent {{ parent }}, child {{ child }}, origin xyz={{ xyz[0] }} {{ xyz[1] }} {{ xyz[2] }} rpy={{ rpy[0] }} {{ rpy[1] }} {{ rpy[2] }}, axis {{ axis[0] }} {{ axis[1] }} {{ axis[2] }}, limit effort={{ servo.effort }} velocity={{ servo.velocity }}
